Commit message: odometry working with ekf

File: CRAP_sim_def/urdf/CRAP.xacro (robot description, xacro)
@@ -1,20 +1,12 @@
 <?xml version="1.0"?>
 <robot xmlns:xacro="http://www.ros.org/wiki/xacro" name="CRAP">
+  <xacro:property name="base_width" value="0.5"/>
+  <xacro:property name="base_length" value="0.5"/>
+  <xacro:property name="base_height" value="0.05"/>
+  <xacro:property name="wheel_radius" value="0.05"/>
+  <xacro:property name="wheel_width" value="0.02"/>
+  <xacro:property name="wheel_ygap" value="0.025"/>
+  <xacro:property name="wheel_zoff" value="0.05"/>
   <!-- Define the base link of the robot -->
-    <link name="base_footprint">
-      <visual>
-          <origin xyz="0 0 0" rpy="0 0 0" />
-          <geometry>
-              <box size="0.001 0.001 0.001" />
-          </geometry>
-      </visual>
-  </link>
-  <gazebo reference="base_footprint">
-      <turnGravityOff>false</turnGravityOff>
-  </gazebo>
-  <joint name="base_footprint_joint" type="fixed">
-      <parent link="base_footprint"/>
-      <child link="base_link" />
-  </joint>
   <link name="base_link">
     <inertial>
@@ -24,7 +16,6 @@
     </inertial>
     <visual>
-      <origin xyz="0 0 0" rpy="0 0 0"/>
       <geometry>
-        <box size="0.5 0.5 0.05"/>
+        <box size="${base_length} ${base_width} ${base_height}"/>
       </geometry>
       <material name="red">
@@ -38,11 +29,20 @@
     </collision>
   </link>
+  <link name="base_footprint"/>
+  <!-- <gazebo reference="base_footprint">
+      <turnGravityOff>false</turnGravityOff>
+  </gazebo> -->
+  <joint name="base_joint" type="fixed">
+    <parent link="base_link"/>
+    <child link="base_footprint"/>
+    <origin xyz="0.0 0.0 ${-(wheel_radius+wheel_zoff)}" rpy="0 0 0"/>
+  </joint>
   <!-- Define the four  wheels -->
   <xacro:include filename="wheel.xacro"/>
-  <xacro:wheel name="front_left_wheel" parent="base_link" x="0.25" y="0.25" />
-  <xacro:wheel name="front_right_wheel" parent="base_link" x="0.25" y="-0.25" />
+  <xacro:wheel name="front_left_wheel" parent="base_link" x="0.25" y="0.25" z = "${-wheel_zoff}" radius = "${wheel_radius}" thickness = "${wheel_width}"/>
+  <xacro:wheel name="front_right_wheel" parent="base_link" x="0.25" y="-0.25" z = "${-wheel_zoff}" radius = "${wheel_radius}" thickness = "${wheel_width}"/>
   <xacro:include filename="wheel_driven.xacro"/>
-  <xacro:wheel_driven name="rear_left_wheel" parent="base_link" x="-0.25" y="0.25" />
-  <xacro:wheel_driven name="rear_right_wheel" parent="base_link" x="-0.25" y="-0.25" />
+  <xacro:wheel_driven name="rear_left_wheel" parent="base_link" x="-0.25" y="0.25" z = "${-wheel_zoff}" radius = "${wheel_radius}" thickness = "${wheel_width}"/>
+  <xacro:wheel_driven name="rear_right_wheel" parent="base_link" x="-0.25" y="-0.25" z = "${-wheel_zoff}" radius = "${wheel_radius}" thickness = "${wheel_width}"/>
   <!-- Define the LIDAR sensor -->
   <xacro:include filename="lidar_gazebo.xacro"/>

File: CRAP_sim_def/urdf/kinect_gazebo.xacro (robot description, xacro)
@@ -7,12 +7,12 @@
             <origin xyz="0 0 0" rpy="0 0 0"/>
             <visual>
-                <origin xyz="0 0 0" rpy="0 0 ${M_PI/2}"/>
+                <origin xyz="0 0 0" rpy="0 0 0"/>
                 <geometry>
-                    <box size="0.15 0.04 0.04" />
+                    <box size="0.04 0.15 0.04" />
                 </geometry>
             </visual>
             <collision>
                 <geometry>
-                    <box size="0.07 0.3 0.09"/>
+                    <box size="0.04 0.15 0.04"/>
                 </geometry>
             </collision>
@@ -25,5 +25,5 @@
         <link name="${prefix}_depth_frame"/>
         <joint name="${prefix}_depth_joint" type="fixed">
-            <origin xyz="0 0 0" rpy="0 0 0"/>
+            <origin xyz="0 0 0" rpy="${-pi/2} 0 ${-pi/2}"/>
             <parent link="${prefix}_link"/>
             <child link="${prefix}_depth_frame"/>
@@ -32,5 +32,5 @@
             <sensor name="depth_camera" type="depth">
                 <visualize>true</visualize>
-                <update_rate>30.0</update_rate>
+                <update_rate>15.0</update_rate>
                 <camera name="kinect">
                 <horizontal_fov>1.047198</horizontal_fov>
@@ -48,5 +48,5 @@
                 <baseline>0.2</baseline>
                 <alwaysOn>true</alwaysOn>
-                <updateRate>0.0</updateRate>
+                <updateRate>15.0</updateRate>
                 <frame_name>camera_depth_frame</frame_name>
                 <pointCloudCutoff>0.5</pointCloudCutoff>

File: CRAP_sim_def/urdf/wheel.xacro (robot description, xacro)
@@ -2,7 +2,7 @@
 <robot xmlns:xacro="http://www.ros.org/wiki/xacro" name="wheel_macro">
   <xacro:property name="M_PI" value="3.141592653589793"/>
-  <xacro:property name="radius" value="0.05"/>
-  <xacro:property name="thickness" value="0.02"/>
-  <xacro:macro name="wheel" params="name parent x y">
+  <!-- <xacro:property name="radius" value="0.05"/>
+  <xacro:property name="thickness" value="0.02"/> -->
+  <xacro:macro name="wheel" params="name parent x y z radius thickness">
     <!-- Define the wheel link -->
     <link name="${name}_link">
@@ -38,5 +38,5 @@
     </joint> -->
     <joint name="${name}_joint" type="fixed">
-      <origin xyz="${x} ${y} 0" rpy="0 0 0"/>
+      <origin xyz="${x} ${y} ${z}" rpy="0 0 0"/>
       <parent link="${parent}"/>
       <child link="${name}_link"/>

File: CRAP_sim_def/urdf/wheel_driven.xacro (robot description, xacro)
@@ -2,7 +2,7 @@
 <robot xmlns:xacro="http://www.ros.org/wiki/xacro" name="wheel_driven">
   <xacro:property name="M_PI" value="3.141592653589793"/>
-  <xacro:property name="radius" value="0.05"/>
-  <xacro:property name="thickness" value="0.02"/>
-  <xacro:macro name="wheel_driven" params="name parent x y">
+  <!-- <xacro:property name="radius" value="0.05"/>
+  <xacro:property name="thickness" value="0.02"/> -->
+  <xacro:macro name="wheel_driven" params="name parent x y z radius thickness">
     <!-- Define the wheel link -->
     <link name="${name}_link">
@@ -30,5 +30,5 @@
     <!-- Define the wheel joint -->
     <joint name="${name}_joint" type="continuous">
-      <origin xyz="${x} ${y} 0" rpy="0 0 0"/>
+      <origin xyz="${x} ${y} ${z}" rpy="0 0 0"/>
       <parent link="${parent}"/>
       <child link="${name}_link"/>

Commit message: Use ROS2_Controller instead of gazebo plugin

File: CRAP_sim_def/urdf/CRAP.xacro (robot description, xacro)
@@ -54,25 +54,40 @@
   <xacro:include filename="imu.xacro"/>
   <xacro:imu prefix="imu" parent="base_link" x="-0.2" y="0" z="0.02"/>
+  <ros2_control name = "GazeboSystem" type = "system">
+    <hardware>
+        <plugin>gazebo_ros2_control/GazeboSystem</plugin>
+    </hardware>
+    <joint name="rear_left_wheel_joint">
+            <command_interface name="velocity">
+                <param name="min">-10</param>
+                <param name="max">10</param>
+            </command_interface>
+            <state_interface name="velocity"/>
+            <state_interface name="position"/>
+    </joint>
+    <joint name="rear_right_wheel_joint">
+        <command_interface name="velocity">
+            <param name="min">-10</param>
+            <param name="max">10</param>
+        </command_interface>
+        <state_interface name="velocity"/>
+        <state_interface name="position"/>
+    </joint>
+  </ros2_control>
   <gazebo>
+    <plugin name="gazebo_ros2_control" filename="libgazebo_ros2_control.so">
+      <parameters>$(find CRAP_sim_def)/config/controller.yaml</parameters>
+    </plugin>
+  </gazebo>
+  <!-- <gazebo>
       <plugin name='diff_drive' filename='libgazebo_ros_diff_drive.so'>
-      <!-- Update rate -->
       <update_rate>100</update_rate>
-      <!-- Number of wheel pairs -->
       <num_wheel_pairs>1</num_wheel_pairs>
-      <!-- wheels0 -->
-      <!-- <left_joint>front_left_wheel_joint</left_joint>
-      <right_joint>front_right_wheel_joint</right_joint> -->
-      <!-- wheels1-->
       <left_joint>rear_left_wheel_joint</left_joint>
       <right_joint>rear_right_wheel_joint</right_joint>
-      <!-- kinematics -->
       <wheel_separation>0.5</wheel_separation>
-      <!-- <wheel_separation>0.5</wheel_separation> -->
       <wheel_diameter>0.1</wheel_diameter>
-      <!-- <wheel_diameter>0.1</wheel_diameter> -->
-      <!-- limits -->
       <max_wheel_torque>20</max_wheel_torque>
       <max_wheel_acceleration>1.0</max_wheel_acceleration>
-      <!-- output -->
       <publish_odom>true</publish_odom>
       <publish_odom_tf>false</publish_odom_tf>
@@ -81,4 +96,4 @@
       <robot_base_frame>base_link</robot_base_frame>
       </plugin>
-  </gazebo>
+  </gazebo> -->
 </robot>

File: CRAP_sim_def/urdf/lidar_gazebo.xacro (robot description, xacro)
@@ -51,5 +51,5 @@
             <range>
                 <min>0.120000</min>
-                <max>3.5</max>
+                <max>8</max>
                 <resolution>0.015000</resolution>
             </range>

File: CRAP_sim_def/urdf/wheel.xacro (robot description, xacro)
@@ -46,6 +46,6 @@
       <kp>1000000.0</kp> <!-- kp and kd for rubber -->
       <kd>100.0</kd>
-      <mu1>0.1</mu1>
-      <mu2>0.1</mu2>
+      <mu1>0.01</mu1>
+      <mu2>0.01</mu2>
       <maxVel>1.0</maxVel>
       <minDepth>0.00</minDepth>

Commit message: minor bug fixes

File: CRAP_sim_def/urdf/CRAP.xacro (robot description, xacro)
@@ -10,9 +10,9 @@
   <!-- Define the base link of the robot -->
   <link name="base_link">
-    <inertial>
+    <!-- <inertial>
       <mass value="10"/>
       <origin xyz="0 0 0" rpy="0 0 0"/>
       <inertia ixx="0.1" ixy="0" ixz="0" iyy="0.1" iyz="0" izz="0.1"/>
-    </inertial>
+    </inertial> -->
     <visual>
       <geometry>
@@ -29,8 +29,20 @@
     </collision>
   </link>
+  <link name="base_link_intertia">
+    <inertial>
+      <mass value="10"/>
+      <origin xyz="0 0 0" rpy="0 0 0"/>
+      <inertia ixx="0.1" ixy="0" ixz="0" iyy="0.1" iyz="0" izz="0.1"/>
+    </inertial>
+  </link>
   <link name="base_footprint"/>
   <!-- <gazebo reference="base_footprint">
       <turnGravityOff>false</turnGravityOff>
   </gazebo> -->
+  <joint name="base_joint_inertia" type="fixed">
+    <parent link="base_link"/>
+    <child link="base_link_intertia"/>
+    <origin xyz="0.0 0.0 0.0" rpy="0 0 0"/>
+  </joint>
   <joint name="base_joint" type="fixed">
     <parent link="base_link"/>

Commit message: added lidar driver ros node

File: CRAP_sim_def/urdf/CRAP.xacro (robot description, xacro)
@@ -62,5 +62,5 @@
   <!-- Define the rgbd camera -->
   <xacro:include filename="kinect_gazebo.xacro"/>
-  <xacro:kinect_camera prefix="kinect" parent="base_link" x="0.27" y="0" z="0"/>
+  <xacro:kinect_camera prefix="kinect2" parent="base_link" x="0.27" y="0" z="0"/>
   <!-- Define the imu camera -->
   <xacro:include filename="imu.xacro"/>

File: CRAP_sim_def/urdf/kinect_gazebo.xacro (robot description, xacro)
@@ -18,4 +18,5 @@
             </collision>
         </link>
+        <!-- location of the kinect relative to base -->
         <joint name="${prefix}_joint" type="fixed">
             <origin xyz="${x} ${y} ${z}" rpy="0 0 0"/>
@@ -24,8 +25,16 @@
         </joint>
         <link name="${prefix}_depth_frame"/>
+        <!-- location of the depth camera relative to kinect frame -->
         <joint name="${prefix}_depth_joint" type="fixed">
             <origin xyz="0 0 0" rpy="${-pi/2} 0 ${-pi/2}"/>
             <parent link="${prefix}_link"/>
             <child link="${prefix}_depth_frame"/>
+        </joint>
+        <link name="${prefix}_rgb_frame"/>
+        <!-- location of the rgb frame relative to kinect frame -->
+        <joint name="${prefix}_rgb_joint" type="fixed">
+            <origin xyz="0 0 0" rpy="${-pi/2} 0 ${-pi/2}"/>
+            <parent link="${prefix}_link"/>
+            <child link="${prefix}_rgb_frame"/>
         </joint>
         <gazebo reference="${prefix}_link">
