Commit message: updated lidar/ros2 control hardware driver

File: CRAP_sim_def/urdf/CRAP_real.xacro (robot description, xacro)
@@ -63,49 +63,6 @@
   <xacro:include filename="kinect_gazebo.xacro"/>
   <xacro:kinect_camera prefix="kinect2" parent="base_link" x="0.27" y="0" z="0"/>
-  <!-- Define the imu camera -->
-  <!-- <xacro:include filename="imu.xacro"/>
-  <xacro:imu prefix="imu" parent="base_link" x="-0.2" y="0" z="0.02"/> -->
-  <ros2_control name = "GazeboSystem" type = "system">
-    <hardware>
-        <plugin>gazebo_ros2_control/GazeboSystem</plugin>
-    </hardware>
-    <joint name="rear_left_wheel_joint">
-            <command_interface name="velocity">
-                <param name="min">-10</param>
-                <param name="max">10</param>
-            </command_interface>
-            <state_interface name="velocity"/>
-            <state_interface name="position"/>
-    </joint>
-    <joint name="rear_right_wheel_joint">
-        <command_interface name="velocity">
-            <param name="min">-10</param>
-            <param name="max">10</param>
-        </command_interface>
-        <state_interface name="velocity"/>
-        <state_interface name="position"/>
-    </joint>
-  </ros2_control>
-  <gazebo>
-    <plugin name="gazebo_ros2_control" filename="libgazebo_ros2_control.so">
-      <parameters>$(find CRAP_sim_def)/config/controller.yaml</parameters>
-    </plugin>
-  </gazebo>
-  <!-- <gazebo>
-      <plugin name='diff_drive' filename='libgazebo_ros_diff_drive.so'>
-      <update_rate>100</update_rate>
-      <num_wheel_pairs>1</num_wheel_pairs>
-      <left_joint>rear_left_wheel_joint</left_joint>
-      <right_joint>rear_right_wheel_joint</right_joint>
-      <wheel_separation>0.5</wheel_separation>
-      <wheel_diameter>0.1</wheel_diameter>
-      <max_wheel_torque>20</max_wheel_torque>
-      <max_wheel_acceleration>1.0</max_wheel_acceleration>
-      <publish_odom>true</publish_odom>
-      <publish_odom_tf>false</publish_odom_tf>
-      <publish_wheel_tf>true</publish_wheel_tf>
-      <odometry_frame>odom</odometry_frame>
-      <robot_base_frame>base_link</robot_base_frame>
-      </plugin>
-  </gazebo> -->
+  <!-- Define ROS2 control -->
+  <xacro:include filename="ros2_control_real.xacro"/>
+  <xacro:diffbot_ros2_control name="DiffBot" prefix="rear_" />
 </robot>

File: CRAP_sim_def/urdf/kinect_gazebo.xacro (robot description, xacro)
@@ -24,17 +24,17 @@
             <child link="${prefix}_link"/>
         </joint>
-        <link name="${prefix}_depth_frame"/>
+        <link name="${prefix}_ir_optical_frame"/>
         <!-- location of the depth camera relative to kinect frame -->
         <joint name="${prefix}_depth_joint" type="fixed">
-            <origin xyz="0 0 0" rpy="${-pi/2} 0 ${-pi/2}"/>
+            <origin xyz="0.03 0 0.045" rpy="${-pi/2} 0 ${-pi/2}"/>
             <parent link="${prefix}_link"/>
-            <child link="${prefix}_depth_frame"/>
+            <child link="${prefix}_ir_optical_frame"/>
         </joint>
-        <link name="${prefix}_rgb_frame"/>
+        <link name="${prefix}_rgb_optical_frame"/>
         <!-- location of the rgb frame relative to kinect frame -->
         <joint name="${prefix}_rgb_joint" type="fixed">
-            <origin xyz="0 0 0" rpy="${-pi/2} 0 ${-pi/2}"/>
+            <origin xyz="0.03 -0.09 0.045" rpy="${-pi/2} 0 ${-pi/2}"/>
             <parent link="${prefix}_link"/>
-            <child link="${prefix}_rgb_frame"/>
+            <child link="${prefix}_rgb_optical_frame"/>
         </joint>
         <gazebo reference="${prefix}_link">
@@ -58,5 +58,5 @@
                 <alwaysOn>true</alwaysOn>
                 <updateRate>15.0</updateRate>
-                <frame_name>${prefix}_depth_frame</frame_name>
+                <frame_name>${prefix}_ir_optical_frame</frame_name>
                 <pointCloudCutoff>0.5</pointCloudCutoff>
                 <pointCloudCutoffMax>3.0</pointCloudCutoffMax>

Commit message: ROS2 control works now with hardware

File: CRAP_sim_def/urdf/CRAP_real.xacro (robot description, xacro)
@@ -65,4 +65,4 @@
   <!-- Define ROS2 control -->
   <xacro:include filename="ros2_control_real.xacro"/>
-  <xacro:diffbot_ros2_control name="DiffBot" prefix="rear_" />
+  <xacro:diffbot_ros2_control name="DiffBot"/>
 </robot>

File: CRAP_sim_def/urdf/ros2_control_real.xacro (robot description, xacro)
@@ -1,14 +1,14 @@
 <?xml version="1.0"?>
 <robot xmlns:xacro="http://www.ros.org/wiki/xacro">
-  <xacro:macro name="diffbot_ros2_control" params="name prefix">
+  <xacro:macro name="diffbot_ros2_control" params="name">
     <ros2_control name="${name}" type="system">
       <hardware>
         <plugin>diffdrive_arduino/DiffDriveArduinoHardware</plugin>
-        <param name="left_wheel_name">left_wheel_joint</param>
-        <param name="right_wheel_name">right_wheel_joint</param>
+        <param name="left_wheel_name">rear_left_wheel_joint</param>
+        <param name="right_wheel_name">rear_right_wheel_joint</param>
         <param name="loop_rate">30</param>
         <param name="device">/dev/ttyACM0</param>
         <param name="baud_rate">57600</param>
-        <param name="timeout_ms">1000</param>
+        <param name="timeout_ms">3000</param>
         <param name="enc_counts_per_rev">9600</param>
         <param name="pid_p">20</param>
@@ -17,10 +17,10 @@
         <param name="pid_o">50</param>
       </hardware>
-      <joint name="${prefix}left_wheel_joint">
+      <joint name="rear_left_wheel_joint">
         <command_interface name="velocity"/>
         <state_interface name="position"/>
         <state_interface name="velocity"/>
       </joint>
-      <joint name="${prefix}right_wheel_joint">
+      <joint name="rear_right_wheel_joint">
         <command_interface name="velocity"/>
         <state_interface name="position"/>

Commit message: updated urdf to reflect real bot

File: CRAP_sim_def/urdf/CRAP_real.xacro (robot description, xacro)
@@ -1,11 +1,11 @@
 <?xml version="1.0"?>
 <robot xmlns:xacro="http://www.ros.org/wiki/xacro" name="CRAP">
-  <xacro:property name="base_width" value="0.5"/>
-  <xacro:property name="base_length" value="0.5"/>
-  <xacro:property name="base_height" value="0.05"/>
-  <xacro:property name="wheel_radius" value="0.05"/>
-  <xacro:property name="wheel_width" value="0.02"/>
+  <xacro:property name="base_width" value="0.265"/>
+  <xacro:property name="base_length" value="0.415"/>
+  <xacro:property name="base_height" value="0.18"/>
+  <xacro:property name="wheel_radius" value="0.051"/>
+  <xacro:property name="wheel_width" value="0.025"/>
   <xacro:property name="wheel_ygap" value="0.025"/>
-  <xacro:property name="wheel_zoff" value="0.05"/>
+  <xacro:property name="wheel_zoff" value="${base_height/2}"/>
   <!-- Define the base link of the robot -->
   <link name="base_link">
@@ -25,5 +25,5 @@
     <collision>
       <geometry>
-          <box size="0.5 0.5 0.05"/>
+          <box size="0.5 0.5 ${base_height}"/>
       </geometry>
     </collision>
@@ -52,15 +52,15 @@
   <!-- Define the four  wheels -->
   <xacro:include filename="wheel.xacro"/>
-  <xacro:wheel name="front_left_wheel" parent="base_link" x="0.25" y="0.25" z = "${-wheel_zoff}" radius = "${wheel_radius}" thickness = "${wheel_width}"/>
-  <xacro:wheel name="front_right_wheel" parent="base_link" x="0.25" y="-0.25" z = "${-wheel_zoff}" radius = "${wheel_radius}" thickness = "${wheel_width}"/>
+  <xacro:wheel name="front_left_wheel" parent="base_link" x="${base_length/2}" y="${(base_width+wheel_width)/2}" z = "${-wheel_zoff}" radius = "${wheel_radius}" thickness = "${wheel_width}"/>
+  <xacro:wheel name="front_right_wheel" parent="base_link" x="${base_length/2}" y="${-(base_width+wheel_width)/2}" z = "${-wheel_zoff}" radius = "${wheel_radius}" thickness = "${wheel_width}"/>
   <xacro:include filename="wheel_driven.xacro"/>
-  <xacro:wheel_driven name="rear_left_wheel" parent="base_link" x="-0.25" y="0.25" z = "${-wheel_zoff}" radius = "${wheel_radius}" thickness = "${wheel_width}"/>
-  <xacro:wheel_driven name="rear_right_wheel" parent="base_link" x="-0.25" y="-0.25" z = "${-wheel_zoff}" radius = "${wheel_radius}" thickness = "${wheel_width}"/>
+  <xacro:wheel_driven name="rear_left_wheel" parent="base_link" x="${-base_length/2}" y="${(base_width+wheel_width)/2}" z = "${-wheel_zoff}" radius = "${wheel_radius}" thickness = "${wheel_width}"/>
+  <xacro:wheel_driven name="rear_right_wheel" parent="base_link" x="${-base_length/2}" y="${-(base_width+wheel_width)/2}" z = "${-wheel_zoff}" radius = "${wheel_radius}" thickness = "${wheel_width}"/>
   <!-- Define the LIDAR sensor -->
   <xacro:include filename="lidar_gazebo.xacro"/>
-  <xacro:rplidar prefix="lidar" parent="base_link" x="0.27" y="0" z="0.1"/>
+  <xacro:rplidar prefix="lidar" parent="base_link" x="0.205" y="0" z="${0.37-base_height/2}"/>
   <!-- Define the rgbd camera -->
   <xacro:include filename="kinect_gazebo.xacro"/>
-  <xacro:kinect_camera prefix="kinect2" parent="base_link" x="0.27" y="0" z="0"/>
+  <xacro:kinect_camera prefix="kinect2" parent="base_link" x="0.205" y="0" z="${0.26-base_height/2}"/>
   <!-- Define ROS2 control -->
   <xacro:include filename="ros2_control_real.xacro"/>

Commit message: change frame names

File: CRAP_sim_def/urdf/CRAP_real.xacro (robot description, xacro)
@@ -62,5 +62,5 @@
   <!-- Define the rgbd camera -->
   <xacro:include filename="kinect_gazebo.xacro"/>
-  <xacro:kinect_camera prefix="kinect2" parent="base_link" x="0.205" y="0" z="${0.26-base_height/2}"/>
+  <xacro:kinect_camera prefix="oak_d" parent="base_link" x="0.205" y="0" z="${0.26-base_height/2}"/>
   <!-- Define ROS2 control -->
   <xacro:include filename="ros2_control_real.xacro"/>

File: CRAP_sim_def/urdf/kinect_gazebo.xacro (robot description, xacro)
@@ -24,7 +24,7 @@
             <child link="${prefix}_link"/>
         </joint>
-        <link name="${prefix}_ir_optical_frame"/>
+        <!-- <link name="${prefix}_ir_optical_frame"/> -->
         <!-- location of the depth camera relative to kinect frame -->
-        <joint name="${prefix}_depth_joint" type="fixed">
+        <!-- <joint name="${prefix}_depth_joint" type="fixed">
             <origin xyz="0.03 0 0.045" rpy="${-pi/2} 0 ${-pi/2}"/>
             <parent link="${prefix}_link"/>
@@ -37,5 +37,5 @@
             <parent link="${prefix}_link"/>
             <child link="${prefix}_rgb_optical_frame"/>
-        </joint>
+        </joint> -->
         <gazebo reference="${prefix}_link">
             <sensor name="depth_camera" type="depth">
