Commit message: rpi

File: CRAP_sim_def/urdf/kinect_gazebo.xacro (robot description, xacro)
@@ -4,5 +4,5 @@
     <xacro:macro name="kinect_camera" params="prefix parent x y z">
         <!-- Create kinect reference frame -->
-        <link name="${prefix}_link">
+        <link name="${prefix}_base_link">
             <origin xyz="0 0 0" rpy="0 0 0"/>
             <visual>
@@ -19,23 +19,17 @@
         </link>
         <!-- location of the kinect relative to base -->
-        <joint name="${prefix}_joint" type="fixed">
+        <joint name="${prefix}_base_joint" type="fixed">
             <origin xyz="${x} ${y} ${z}" rpy="0 0 0"/>
             <parent link="${parent}"/>
+            <child link="${prefix}_base_link"/>
+        </joint>
+        <link name="${prefix}_link"/>
+        <!-- location of the depth camera relative to kinect frame -->
+       <joint name="${prefix}_joint" type="fixed">
+            <origin xyz="0 0 0" rpy="${pi/2+15/180*pi} 0 ${pi/2}"/>
+            <parent link="${prefix}_base_link"/>
             <child link="${prefix}_link"/>
         </joint>
-        <!-- <link name="${prefix}_ir_optical_frame"/> -->
-        <!-- location of the depth camera relative to kinect frame -->
-        <!-- <joint name="${prefix}_depth_joint" type="fixed">
-            <origin xyz="0.03 0 0.045" rpy="${-pi/2} 0 ${-pi/2}"/>
-            <parent link="${prefix}_link"/>
-            <child link="${prefix}_ir_optical_frame"/>
-        </joint>
-        <link name="${prefix}_rgb_optical_frame"/>
-        <!-- location of the rgb frame relative to kinect frame -->
-        <joint name="${prefix}_rgb_joint" type="fixed">
-            <origin xyz="0.03 -0.09 0.045" rpy="${-pi/2} 0 ${-pi/2}"/>
-            <parent link="${prefix}_link"/>
-            <child link="${prefix}_rgb_optical_frame"/>
-        </joint> -->
+        <!-- <link name="${prefix}_rgb_optical_frame"/>
         <gazebo reference="${prefix}_link">
             <sensor name="depth_camera" type="depth">
@@ -73,5 +67,5 @@
                 </plugin>
             </sensor>
-        </gazebo>
+        </gazebo> -->
     </xacro:macro>
 </robot>
